Commit message: mors meets gym

File: mors_sim/urdf/mors.urdf (robot description, URDF)
Before this commit: robot mors_sim, 21 links, 20 joints
Links:
- removed link scan_frame
- added link head_link, mass 0.5; collision mesh filename=package://mors_sim/urdf/meshes/robohead.stl scale=1 1 1; visual mesh filename=package://mors_sim/urdf/meshes/robohead.stl scale=1 1 1
- added link scan, mass 0.001
Joints:
- added joint head_joint: type fixed, parent base_link, child head_link, origin xyz=0.16 0 0.07 rpy=0 0 0
- joint scan_joint: child scan_frame -> scan; origin xyz=0.15 0.0 0.115 rpy=0 0 0 -> (none)

File: mors_sim/urdf/mors.xacro (robot description, xacro)
@@ -282,7 +282,18 @@
     </inertial>
   </link>
-  <xacro:rplidar_a1 name="scan" topics_ns="scan" parent="base_link">
+  <!-- <xacro:rplidar_a1 name="scan" topics_ns="scan" parent="base_link">
     <origin rpy="0 0 0" xyz="0.15 0.0 0.115"/>
-  </xacro:rplidar_a1>
+  </xacro:rplidar_a1>  -->
+  <link name="scan">
+    <inertial>
+      <mass value="0.001"/>
+      <origin rpy="0 0 0" xyz="0.15 0.0 0.115"/>
+      <inertia ixx="1e-09" ixy="0.0" ixz="0.0" iyy="1e-09" iyz="0.0" izz="1e-09"/>
+    </inertial>
+  </link>
+  <joint name="scan_joint" type="fixed">
+    <parent link="base_link"/>
+    <child link="scan"/>
+  </joint>
   <link name="imu_link">
     <inertial>
@@ -296,3 +307,27 @@
     <child link="imu_link"/>
   </joint>
+  <link name="head_link">
+    <visual>
+      <origin rpy="0 0 0" xyz="0 0 0"/>
+      <geometry>
+        <mesh filename="${mesh_addr}robohead.stl" scale="1 1 1"/>
+      </geometry>
+      <material name="silver"/>
+    </visual>
+    <collision>
+      <geometry>
+        <mesh filename="${mesh_addr}robohead.stl" scale="1 1 1"/>
+      </geometry>
+    </collision>
+    <inertial>
+      <mass value="0.5"/>
+      <origin rpy="0 0 0" xyz="0.0 0 0.0"/>
+      <inertia ixx="1e-09" ixy="0.0" ixz="0.0" iyy="1e-09" iyz="0.0" izz="1e-09"/>
+    </inertial>
+  </link>
+  <joint name="head_joint" type="fixed">
+    <parent link="base_link"/>
+    <child link="head_link"/>
+    <origin rpy="0 0 0" xyz="0.16 0 0.07"/>
+  </joint>
 </robot>

Commit message: robogui changed

File: mors_sim/urdf/mors.urdf (robot description, URDF)
Before this commit: robot mors_sim, 22 links, 21 joints
Links:
- removed link head_link
Joints:
- removed joint head_joint
